Commit message: Remove oak_imu_frame and oak_imu_joint (OAK-D-LITE has no IMU)

File: lepantilt_description/urdf/pantilt.urdf (robot description, URDF)
Before this commit: robot lepantilt, 13 links, 12 joints
Links:
- removed link oak_imu_frame
Joints:
- removed joint oak_imu_joint

File: lepantilt_description/urdf/pantilt.urdf.xacro (robot description, xacro)
@@ -126,11 +126,4 @@
     cam_roll="${oak_roll}" cam_pitch="0" cam_yaw="${oak_yaw}"
     r="0.15" g="0.15" b="0.15" a="1.0"/>
-  <!-- OAK-D-S2 IMU frame (hardcoded until upstream depthai_descriptions adds OAK-D-S2 IMU support) -->
-  <link name="oak_imu_frame"/>
-  <joint name="oak_imu_joint" type="fixed">
-    <parent link="oak"/>
-    <child link="oak_imu_frame"/>
-    <origin xyz="-0.008 -0.037945 -0.00079" rpy="${pi} ${pi/2} 0"/>
-  </joint>
   <!-- ROS 2 CONTROL -->
   <ros2_control name="lepantilt_control" type="system">

Commit message: Rename oak_d_s2.stl -> oakd_s2.stl; add oak_imu_frame and oak_imu_joint

File: lepantilt_description/urdf/pantilt.urdf (robot description, URDF)
Before this commit: robot lepantilt, 12 links, 11 joints
Links:
- added link oak_imu_frame
- link oak_model_origin: geometry visual mesh filename=../meshes/oakd_s2.stl
Joints:
- added joint oak_imu_joint: type fixed, parent oak, child oak_imu_frame, origin xyz=-0.008 -0.037945 -0.00079 rpy=3.1415926535897932 1.5707963267948966 0.0

File: lepantilt_description/urdf/pantilt.urdf.xacro (robot description, xacro)
@@ -126,4 +126,11 @@
     cam_roll="${oak_roll}" cam_pitch="0" cam_yaw="${oak_yaw}"
     r="0.15" g="0.15" b="0.15" a="1.0"/>
+  <!-- OAK-D-S2 IMU frame -->
+  <link name="oak_imu_frame"/>
+  <joint name="oak_imu_joint" type="fixed">
+    <parent link="oak"/>
+    <child link="oak_imu_frame"/>
+    <origin xyz="-0.008 -0.037945 -0.00079" rpy="${pi} ${pi/2} 0"/>
+  </joint>
   <!-- ROS 2 CONTROL -->
   <ros2_control name="lepantilt_control" type="system">
