Commit message: Move oak_imu offsets to pantilt.common.xacro

File: lepantilt_description/urdf/pantilt.common.xacro (robot description, xacro)
@@ -30,3 +30,9 @@
   <xacro:property name="oak_roll" value="${-pi/2}"/>
   <xacro:property name="oak_yaw"  value="${-pi/2}"/>
+  <!-- OAK-D-S2 IMU offset (relative to oak frame) -->
+  <xacro:property name="oak_imu_x" value="-0.008"/>
+  <xacro:property name="oak_imu_y" value="-0.037945"/>
+  <xacro:property name="oak_imu_z" value="-0.00079"/>
+  <xacro:property name="oak_imu_r" value="${pi}"/>
+  <xacro:property name="oak_imu_p" value="${pi/2}"/>
 </robot>

File: lepantilt_description/urdf/pantilt.urdf.xacro (robot description, xacro)
@@ -131,5 +131,5 @@
     <parent link="oak"/>
     <child link="oak_imu_frame"/>
-    <origin xyz="-0.008 -0.037945 -0.00079" rpy="${pi} ${pi/2} 0"/>
+    <origin xyz="${oak_imu_x} ${oak_imu_y} ${oak_imu_z}" rpy="${oak_imu_r} ${oak_imu_p} 0"/>
   </joint>
   <!-- ROS 2 CONTROL -->

Commit message: Use charcoal_r/g/b/a properties for depthai_camera color instead of hardcoded values

File: lepantilt_description/urdf/pantilt.common.xacro (robot description, xacro)
@@ -4,4 +4,8 @@
   <xacro:property name="light_grey_rgba" value="0.8 0.8 0.8 1.0"/>
   <xacro:property name="charcoal_rgba" value="0.15 0.15 0.15 1.0"/>
+  <xacro:property name="charcoal_r" value="0.15"/>
+  <xacro:property name="charcoal_g" value="0.15"/>
+  <xacro:property name="charcoal_b" value="0.15"/>
+  <xacro:property name="charcoal_a" value="1.0"/>
   <!-- Pantilt base visual compensation / mount rotation (rad) -->
   <xacro:property name="pantilt_offset_rz" value="${pi/2}"/>

File: lepantilt_description/urdf/pantilt.urdf.xacro (robot description, xacro)
@@ -125,5 +125,5 @@
     cam_pos_x="${oak_pos_x}" cam_pos_y="${oak_pos_y}" cam_pos_z="0"
     cam_roll="${oak_roll}" cam_pitch="0" cam_yaw="${oak_yaw}"
-    r="0.15" g="0.15" b="0.15" a="1.0"/>
+    r="${charcoal_r}" g="${charcoal_g}" b="${charcoal_b}" a="${charcoal_a}"/>
   <!-- OAK-D-S2 IMU frame -->
   <link name="oak_imu_frame"/>

Commit message: clean up + tested code

File: lepantilt_description/urdf/pantilt.common.xacro (robot description, xacro)
@@ -4,8 +4,5 @@
   <xacro:property name="light_grey_rgba" value="0.8 0.8 0.8 1.0"/>
   <xacro:property name="charcoal_rgba" value="0.15 0.15 0.15 1.0"/>
-  <xacro:property name="charcoal_r" value="0.15"/>
-  <xacro:property name="charcoal_g" value="0.15"/>
-  <xacro:property name="charcoal_b" value="0.15"/>
-  <xacro:property name="charcoal_a" value="1.0"/>
+  <xacro:property name="charcoal_rgb" value="0.15"/>
   <!-- Pantilt base visual compensation / mount rotation (rad) -->
   <xacro:property name="pantilt_offset_rz" value="${pi/2}"/>

File: lepantilt_description/urdf/pantilt.control.xacro (robot description, xacro)
@@ -1,21 +1,22 @@
 <?xml version="1.0"?>
 <robot xmlns:xacro="http://www.ros.org/wiki/xacro">
-  <!-- Arguments (externally settable via command line) -->
-  <xacro:arg name="serial_port"    default="/dev/ttySERVO"/>
-  <xacro:arg name="baud_rate"      default="1000000"/>
-  <xacro:arg name="use_mock"       default="false"/>
-  <xacro:arg name="use_sync_write" default="true"/>
-  <!-- Pantilt motor IDs and mode -->
-  <xacro:property name="pan_motor_id" value="1"/>
-  <xacro:property name="tilt_motor_id" value="2"/>
-  <xacro:property name="pantilt_operating_mode" value="0"/>  <!-- Position mode -->
+  <!-- Arguments (externally settable) -->
+  <xacro:arg name="serial_port"       default="/dev/ttyACM0"/>
+  <xacro:arg name="baud_rate"         default="1000000"/>
+  <xacro:arg name="use_mock"          default="false"/>
+  <xacro:arg name="use_sync_write"    default="true"/>
+  <xacro:arg name="pan_motor_id"      default="1"/>
+  <xacro:arg name="tilt_motor_id"     default="2"/>
+  <xacro:arg name="pan_center_steps"  default="2048"/>
+  <xacro:arg name="tilt_center_steps" default="2048"/>
   <!-- Motor-specific parameter (STS3215 default) -->
-  <xacro:property name="sts_max_velocity_steps" value="3400"/>  <!-- Max hardware velocity in steps/s -->
-  <!-- Maximum allowable torque/velocity for each motor -->
-  <xacro:property name="max_velocity_rads" value="${sts_max_velocity_steps*2*pi/4096}"/>  <!-- rad/s -->
+  <xacro:property name="pantilt_operating_mode" default="0"/>  <!-- Position mode -->
+  <xacro:property name="sts_max_velocity_steps" value="3400"/>  <!-- Max hardware velocity in steps/s (absolute motor limit, do not exceed) -->
+  <xacro:property name="max_velocity_steps" value="${int(sts_max_velocity_steps * 0.5)}"/> <!-- steps/second (85% of hardware max, 15% safety margin) -->
+  <xacro:property name="max_velocity_rads" value="${max_velocity_steps*2*pi/4096}"/> <!-- rad/s -->
   <xacro:property name="max_torque_nm" value="2.942"/>  <!-- N⋅m (30 kgf⋅cm for STS3215) -->
   <!-- Pan and Tilt joint limits -->
-  <xacro:property name="pan_joint_lower" value="-2"/>
-  <xacro:property name="pan_joint_upper" value="2"/>
+  <xacro:property name="pan_joint_lower" value="${-pi/2}"/>
+  <xacro:property name="pan_joint_upper" value="${pi/2}"/>
   <xacro:property name="tilt_joint_lower" value="${-pi/2}"/>
   <xacro:property name="tilt_joint_upper" value="${pi/2}"/>
@@ -34,10 +35,10 @@
     <!-- Pan axis: rotates the payload around Z (Motor ID ${pan_motor_id}) -->
     <joint name="pan_joint">
-      <param name="motor_id">${pan_motor_id}</param>
+      <param name="motor_id">$(arg pan_motor_id)</param>
       <param name="operating_mode">${pantilt_operating_mode}</param>
       <param name="min_position">${pan_joint_lower}</param>
       <param name="max_position">${pan_joint_upper}</param>
       <param name="max_velocity">${max_velocity_rads}</param>
-      <param name="position_center_steps">2048</param>
+      <param name="position_center_steps">$(arg pan_center_steps)</param>
       <command_interface name="position"/>
       <state_interface name="position"/>
@@ -51,10 +52,10 @@
     <!-- Tilt axis: rotates the payload around Y (Motor ID ${tilt_motor_id}) -->
     <joint name="tilt_joint">
-      <param name="motor_id">${tilt_motor_id}</param>
+      <param name="motor_id">$(arg tilt_motor_id)</param>
       <param name="operating_mode">${pantilt_operating_mode}</param>
       <param name="min_position">${tilt_joint_lower}</param>
       <param name="max_position">${tilt_joint_upper}</param>
       <param name="max_velocity">${max_velocity_rads}</param>
-      <param name="position_center_steps">2048</param>
+      <param name="position_center_steps">$(arg tilt_center_steps)</param>
       <command_interface name="position"/>
       <state_interface name="position"/>

File: lepantilt_description/urdf/pantilt.module.xacro (robot description, xacro)
@@ -1,8 +1,5 @@
 <?xml version="1.0"?>
 <robot xmlns:xacro="http://www.ros.org/wiki/xacro">
-  <!-- Pan-tilt module: mechanical parts only (no ros2_control)
-       Attach to parent platform (e.g., lekiwi base_link) at specified origin -->
   <xacro:include filename="$(find lepantilt_description)/urdf/pantilt.common.xacro"/>
-  <!-- <xacro:include filename="$(find depthai_descriptions)/urdf/include/depthai_macro.urdf.xacro"/> -->
   <xacro:macro name="lepantilt_module" params="parent *origin">
     <!-- Material definitions (referenced by links below) -->
@@ -96,4 +93,10 @@
       </collision>
     </link>
+    <!-- For the Pan and Tilt joints below, velocity="1e6":
+    URDF requires a velocity attribute on revolute joints, but hardware-enforced
+    velocity profiling makes software rate-limiting redundant and causes spurious
+    "command out of limits" errors from ros2_control when joy_teleop sends large absolute
+    position steps. 1e6 rad/s is physically unreachable and effectively disables the
+    JointSaturationLimiter's per-cycle velocity clipping for these joints. -->
     <!-- Pan joint (revolute) -->
     <joint name="pan_joint" type="revolute">
@@ -102,5 +105,5 @@
       <origin xyz="${pan_joint_x} 0 ${pan_joint_z}" rpy="0 0 0"/>
       <axis xyz="0 0 1"/>
-      <limit lower="${pan_joint_lower}" upper="${pan_joint_upper}" effort="${max_torque_nm}" velocity="${max_velocity_rads}"/>
+      <limit lower="${pan_joint_lower}" upper="${pan_joint_upper}" effort="${max_torque_nm}" velocity="1e6"/>
     </joint>
     <!-- Tilt joint (revolute) -->
@@ -109,24 +112,17 @@
       <child link="tilt_link"/>
       <origin xyz="${tilt_joint_x} 0 ${tilt_joint_z}" rpy="${tilt_joint_rx} ${tilt_joint_ry} 0"/>
-      <axis xyz="0 0 1"/>
-      <limit lower="${tilt_joint_lower}" upper="${tilt_joint_upper}" effort="${max_torque_nm}" velocity="${max_velocity_rads}"/>
+      <axis xyz="0 0 -1"/>
+      <limit lower="${tilt_joint_lower}" upper="${tilt_joint_upper}" effort="${max_torque_nm}" velocity="1e6"/>
     </joint>
-    <!-- OAK-D Camera (direct inclusion) -->
-    <xacro:include filename="$(find depthai_descriptions)/urdf/include/depthai_macro.urdf.xacro"/>
-    <xacro:depthai_camera
+    <!-- OAK-D-S2 Camera + IMU -->
+    <xacro:include filename="$(find lepantilt_description)/urdf/oakd_s2.urdf.xacro"/>
+    <xacro:oakd_s2_camera
       camera_name="oak_link"
-      camera_model="OAK-D-S2"
       base_frame="oak_link"
       parent="tilt_link"
       cam_pos_x="${oak_pos_x}" cam_pos_y="${oak_pos_y}" cam_pos_z="0"
       cam_roll="${oak_roll}" cam_pitch="0" cam_yaw="${oak_yaw}"
-      r="${charcoal_r}" g="${charcoal_g}" b="${charcoal_b}" a="1.0"/>
-    <!-- OAK-D-S2 IMU frame -->
-    <link name="oak_imu_frame"/>
-    <joint name="oak_imu_joint" type="fixed">
-      <parent link="oak_link"/>
-      <child link="oak_imu_frame"/>
-      <origin xyz="${oak_imu_x} ${oak_imu_y} ${oak_imu_z}" rpy="${oak_imu_r} ${oak_imu_p} 0"/>
-    </joint>
+      r="${charcoal_rgb}" g="${charcoal_rgb}" b="${charcoal_rgb}" a="1.0"
+      imu_frame="oak_imu_frame"/>
   </xacro:macro>
 </robot>

File: lepantilt_description/urdf/pantilt.urdf (robot description, URDF)
Before this commit: robot lepantilt, 4 links, 3 joints
Links:
- added link oak_imu_frame
- added link oak_link
- added link oak_link_model_origin; visual mesh filename=../meshes/oakd_s2.stl
- link pan_link: geometry collision mesh filename=../meshes/pan_joint.stl; visual mesh filename=../meshes/pan_joint.stl
- link pantilt_base_link: geometry collision mesh filename=../meshes/pantilt_base.stl; visual mesh filename=../meshes/pan_motor.stl
- link tilt_link: geometry collision mesh filename=../meshes/tilt_joint.stl; visual mesh filename=../meshes/tilt_joint.stl
Joints:
- added joint oak_imu_frame_joint: type fixed, parent oak_link, child oak_imu_frame, origin xyz=-0.008 -0.037945 -0.00079 rpy=3.141592653589793 1.5707963267948966 0
- added joint oak_link_center_joint: type fixed, parent tilt_link, child oak_link, origin xyz=-0.03435 -0.01 0 rpy=-1.5707963267948966 0 -1.5707963267948966
- added joint oak_link_model_origin_joint: type fixed, parent oak_link, child oak_link_model_origin, origin xyz=0 0 0 rpy=1.5707963267948966 0 1.5707963267948966
- joint pan_joint: limit lower=-2 upper=2 effort=2.942 velocity=5.21553467881118 -> lower=-1.5707963267948966 upper=1.5707963267948966 effort=2.942 velocity=1e6
- joint tilt_joint: axis 0 0 1 -> 0 0 -1; limit lower=-1.5707963267948966 upper=1.5707963267948966 effort=2.942 velocity=5.21553467881118 -> lower=-1.5707963267948966 upper=1.5707963267948966 effort=2.942 velocity=1e6

File: lepantilt_description/urdf/pantilt.urdf.xacro (robot description, xacro)
@@ -1,9 +1,16 @@
 <?xml version="1.0"?>
 <robot name="lepantilt" xmlns:xacro="http://www.ros.org/wiki/xacro">
+  <xacro:arg name="serial_port"    default="/dev/ttySERVO"/>
+  <xacro:arg name="baud_rate"      default="1000000"/>
+  <xacro:arg name="use_mock"       default="false"/>
+  <xacro:arg name="use_sync_write" default="true"/>
+  <xacro:arg name="pan_motor_id"   default="1"/>
+  <xacro:arg name="tilt_motor_id"  default="2"/>
+  <xacro:arg name="pan_center_steps" default="2048"/>
+  <xacro:arg name="tilt_center_steps" default="2646"/>
+  <xacro:arg name="pantilt_operating_mode" default="0"/>
   <xacro:include filename="$(find lepantilt_description)/urdf/pantilt.common.xacro"/>
   <xacro:include filename="$(find lepantilt_description)/urdf/pantilt.control.xacro"/>
   <xacro:include filename="$(find lepantilt_description)/urdf/pantilt.module.xacro"/>
-  <!-- OAK-D camera and IMU integration -->
-  <xacro:include filename="$(find depthai_descriptions)/urdf/include/depthai_macro.urdf.xacro"/>
   <!-- Standalone pantilt module instantiation -->
   <link name="base_footprint"/>
